File: KiCAD/Church Controller.sch (KiCad schematic (older format))
At the start: 26 parts, among them J1 Battery Connector, J2 Programming, J3 Prog Jumper, SW1 Change, SW2 Save, U1 AZ1117-3.3, U2 ESP-12E

Commit message: Update
Organized schematic
Other:
- note added: "Buttons"
- note added: "ESP12"
- note added: "LEDs"
- note added: "Power"
- note added: "Prog Header"
- note added: "VCC is from 3x AA Batteries for nominal 4.5v"
- note removed: "VCC is from 3x AA Batteries for 4.5v"
- moved on the sheet: U1
