File: KiCAD/Church Controller.sch (KiCad schematic (older format))
At the start: 24 parts, among them J1 Battery Connector, J2 Programming, SW1 Change, SW2 Save, U1 AZ1117-3.3, U2 ESP-12E

Commit message: Correction
I didn't realize that you couldn't use GPIO 9 on the ESP-12e. Moved battery LED to GPIO 13.
Connections:
- wire segments 74 -> 75
- no-connect marks 6 -> 5
Changed lines of the file:
@@
 	1    0    0    -1
 $EndComp
-Text Label 4750 3500 2    50   ~ 0
+Text Label 6400 3400 0    50   ~ 0
 LED_BATT
 Wire Wire Line
@@
 NoConn ~ 5000 3700
 NoConn ~ 5000 3800
-NoConn ~ 6200 3400
 $Comp
 L power:GND #PWR0122
@@
 Wire Wire Line
 	900  4900 1550 4900
+Wire Wire Line
+	6200 3400 6400 3400
 $EndSCHEMATC
