File: KiCAD/_saved_Church Controller.sch (KiCad schematic (older format))
At the start: 24 parts, among them J1 Battery Connector, J2 Programming, SW1 Change, SW2 Save, U1 AZ1117-3.3, U2 ESP-12E

Commit message: Update
Changed programming header, organized silkscreen, generated gerbers, added one missing trace.
Changed lines of the file:
@@
 L Device:LED D1
 U 1 1 5EF550FA
-P 9900 2400
-F 0 "D1" H 9891 2616 50  0000 C CNN
-F 1 "Green" H 9891 2525 50  0000 C CNN
-F 2 "LED_THT:LED_D5.0mm" H 9900 2400 50  0001 C CNN
-F 3 "~" H 9900 2400 50  0001 C CNN
-	1    9900 2400
+P 9900 2150
+F 0 "D1" H 9891 2366 50  0000 C CNN
+F 1 "Green" H 9891 2275 50  0000 C CNN
+F 2 "LED_THT:LED_D5.0mm" H 9900 2150 50  0001 C CNN
+F 3 "~" H 9900 2150 50  0001 C CNN
+	1    9900 2150
 	1    0    0    -1
 $EndComp
@@
 L Device:LED D2
 U 1 1 5EF551AE
-P 9900 2750
-F 0 "D2" H 9891 2966 50  0000 C CNN
-F 1 "Yellow" H 9891 2875 50  0000 C CNN
-F 2 "LED_THT:LED_D5.0mm" H 9900 2750 50  0001 C CNN
-F 3 "~" H 9900 2750 50  0001 C CNN
-	1    9900 2750
+P 9900 2500
+F 0 "D2" H 9891 2716 50  0000 C CNN
+F 1 "Yellow" H 9891 2625 50  0000 C CNN
+F 2 "LED_THT:LED_D5.0mm" H 9900 2500 50  0001 C CNN
+F 3 "~" H 9900 2500 50  0001 C CNN
+	1    9900 2500
 	1    0    0    -1
 $EndComp
@@
 L Device:LED D3
 U 1 1 5EF551E0
-P 9900 3100
-F 0 "D3" H 9891 3316 50  0000 C CNN
-F 1 "Red" H 9891 3225 50  0000 C CNN
-F 2 "LED_THT:LED_D5.0mm" H 9900 3100 50  0001 C CNN
-F 3 "~" H 9900 3100 50  0001 C CNN
-	1    9900 3100
+P 9900 2850
+F 0 "D3" H 9891 3066 50  0000 C CNN
+F 1 "Red" H 9891 2975 50  0000 C CNN
+F 2 "LED_THT:LED_D5.0mm" H 9900 2850 50  0001 C CNN
+F 3 "~" H 9900 2850 50  0001 C CNN
+	1    9900 2850
 	1    0    0    -1
 $EndComp
@@
 L Device:R_Small R5
 U 1 1 5EF55216
-P 9400 2400
-F 0 "R5" V 9204 2400 50  0000 C CNN
-F 1 "R_Small" V 9295 2400 50  0000 C CNN
-F 2 "Resistor_SMD:R_0805_2012Metric_Pad1.15x1.40mm_HandSolder" H 9400 2400 50  0001 C CNN
-F 3 "~" H 9400 2400 50  0001 C CNN
-	1    9400 2400
+P 9400 2150
+F 0 "R5" V 9204 2150 50  0000 C CNN
+F 1 "R_Small" V 9295 2150 50  0000 C CNN
+F 2 "Resistor_SMD:R_0805_2012Metric_Pad1.15x1.40mm_HandSolder" H 9400 2150 50  0001 C CNN
+F 3 "~" H 9400 2150 50  0001 C CNN
+	1    9400 2150
 	0    1    1    0
 $EndComp
@@
 L Device:R_Small R6
 U 1 1 5EF5528B
-P 9400 2750
-F 0 "R6" V 9204 2750 50  0000 C CNN
-F 1 "R_Small" V 9295 2750 50  0000 C CNN
-F 2 "Resistor_SMD:R_0805_2012Metric_Pad1.15x1.40mm_HandSolder" H 9400 2750 50  0001 C CNN
-F 3 "~" H 9400 2750 50  0001 C CNN
-	1    9400 2750
+P 9400 2500
+F 0 "R6" V 9204 2500 50  0000 C CNN
+F 1 "R_Small" V 9295 2500 50  0000 C CNN
+F 2 "Resistor_SMD:R_0805_2012Metric_Pad1.15x1.40mm_HandSolder" H 9400 2500 50  0001 C CNN
+F 3 "~" H 9400 2500 50  0001 C CNN
+	1    9400 2500
 	0    1    1    0
 $EndComp
@@
 L Device:R_Small R7
 U 1 1 5EF552CD
-P 9400 3100
-F 0 "R7" V 9204 3100 50  0000 C CNN
-F 1 "R_Small" V 9295 3100 50  0000 C CNN
-F 2 "Resistor_SMD:R_0805_2012Metric_Pad1.15x1.40mm_HandSolder" H 9400 3100 50  0001 C CNN
-F 3 "~" H 9400 3100 50  0001 C CNN
-	1    9400 3100
+P 9400 2850
+F 0 "R7" V 9204 2850 50  0000 C CNN
+F 1 "R_Small" V 9295 2850 50  0000 C CNN
+F 2 "Resistor_SMD:R_0805_2012Metric_Pad1.15x1.40mm_HandSolder" H 9400 2850 50  0001 C CNN
+F 3 "~" H 9400 2850 50  0001 C CNN
+	1    9400 2850
 	0    1    1    0
 $EndComp
 Wire Wire Line
-	10300 2200 10300 2400
-Wire Wire Line
-	10300 2400 10050 2400
-Wire Wire Line
-	10050 2750 10300 2750
-Wire Wire Line
-	10300 2750 10300 2400
-Connection ~ 10300 2400
-Wire Wire Line
-	10050 3100 10300 3100
-Wire Wire Line
-	10300 3100 10300 2750
-Wire Wire Line
-	9750 2400 9500 2400
-Wire Wire Line
-	9750 2750 9500 2750
-Wire Wire Line
-	9750 3100 9500 3100
-Text Label 9050 2400 2    50   ~ 0
+	10300 1950 10300 2150
+Wire Wire Line
+	10300 2150 10050 2150
+Wire Wire Line
+	10050 2500 10300 2500
+Wire Wire Line
+	10300 2500 10300 2150
+Connection ~ 10300 2150
+Wire Wire Line
+	10050 2850 10300 2850
+Wire Wire Line
+	10300 2850 10300 2500
+Wire Wire Line
+	9750 2150 9500 2150
+Wire Wire Line
+	9750 2500 9500 2500
+Wire Wire Line
+	9750 2850 9500 2850
+Text Label 9050 2150 2    50   ~ 0
 LED_GREEN
-Text Label 9050 2750 2    50   ~ 0
+Text Label 9050 2500 2    50   ~ 0
 LED_YELLOW
-Text Label 9050 3100 2    50   ~ 0
+Text Label 9050 2850 2    50   ~ 0
 LED_RED
 Wire Wire Line
-	9300 2400 9050 2400
-Wire Wire Line
-	9300 2750 9050 2750
-Wire Wire Line
-	9050 3100 9300 3100
+	9300 2150 9050 2150
+Wire Wire Line
+	9300 2500 9050 2500
+Wire Wire Line
+	9050 2850 9300 2850
 Text Label 6400 3300 0    50   ~ 0
 LED_GREEN
@@
 L power:+3V3 #PWR0115
 U 1 1 5EF69FC4
-P 10300 2200
-F 0 "#PWR0115" H 10300 2050 50  0001 C CNN
-F 1 "+3V3" H 10315 2373 50  0000 C CNN
-F 2 "" H 10300 2200 50  0001 C CNN
-F 3 "" H 10300 2200 50  0001 C CNN
-	1    10300 2200
+P 10300 1950
+F 0 "#PWR0115" H 10300 1800 50  0001 C CNN
+F 1 "+3V3" H 10315 2123 50  0000 C CNN
+F 2 "" H 10300 1950 50  0001 C CNN
+F 3 "" H 10300 1950 50  0001 C CNN
+	1    10300 1950
 	1    0    0    -1
 $EndComp
@@
 L power:GND #PWR0117
 U 1 1 5EF76185
-P 1300 4900
-F 0 "#PWR0117" H 1300 4650 50  0001 C CNN
-F 1 "GND" H 1305 4727 50  0000 C CNN
-F 2 "" H 1300 4900 50  0001 C CNN
-F 3 "" H 1300 4900 50  0001 C CNN
-	1    1300 4900
+P 900 4400
+F 0 "#PWR0117" H 900 4150 50  0001 C CNN
+F 1 "GND" H 905 4227 50  0000 C CNN
+F 2 "" H 900 4400 50  0001 C CNN
+F 3 "" H 900 4400 50  0001 C CNN
+	1    900  4400
 	1    0    0    -1
 $EndComp
@@
 Wire Wire Line
 	1300 4600 1550 4600
-Wire Wire Line
-	1300 4900 1550 4900
-Connection ~ 10300 2750
+Connection ~ 10300 2500
 $Comp
 L Device:LED D4
@@
 Wire Wire Line
 	3500 2650 3500 2800
-Wire Wire Line
-	3500 3100 4450 3100
 Connection ~ 3500 3100
 Wire Wire Line
@@
 NoConn ~ 5000 3800
 NoConn ~ 6200 3400
-Wire Wire Line
-	1300 4350 1300 4400
-Wire Wire Line
-	1300 4400 1550 4400
 $Comp
 L power:GND #PWR0122
@@
 Prog Header
 Wire Wire Line
-	4450 2700 4450 3100
-Connection ~ 4450 3100
-Wire Wire Line
-	4450 3100 5000 3100
-Wire Wire Line
 	4450 2150 4450 2500
 Text Label 4950 2700 2    50   ~ 0
@@
 ~RST
 $Comp
-L power:+3V3 #PWR?
+L power:+3V3 #PWR0106
 U 1 1 5F2E2201
-P 1300 4350
-F 0 "#PWR?" H 1300 4200 50  0001 C CNN
-F 1 "+3V3" H 1315 4523 50  0000 C CNN
-F 2 "" H 1300 4350 50  0001 C CNN
-F 3 "" H 1300 4350 50  0001 C CNN
-	1    1300 4350
+P 900 4850
+F 0 "#PWR0106" H 900 4700 50  0001 C CNN
+F 1 "+3V3" H 915 5023 50  0000 C CNN
+F 2 "" H 900 4850 50  0001 C CNN
+F 3 "" H 900 4850 50  0001 C CNN
+	1    900  4850
 	1    0    0    -1
 $EndComp
@@
 Wire Wire Line
 	1300 4800 1550 4800
+Wire Wire Line
+	3500 3100 5000 3100
+Wire Wire Line
+	4450 2700 4450 2900
+Wire Wire Line
+	4450 2900 5000 2900
+Wire Wire Line
+	900  4400 1550 4400
+Wire Wire Line
+	900  4850 900  4900
+Wire Wire Line
+	900  4900 1550 4900
 $EndSCHEMATC
