File: KiCAD/Church Controller.kicad_pcb (KiCad board)
At the start: 2 copper layers, 50 x 90 mm, 26 parts, among them J1 Battery Connector, J2 Programming, J3 Prog Jumper, SW1 Change, SW2 Save, U1 AZ1117-3.3, U2 ESP-12E

Commit message: Update
Changed programming header, organized silkscreen, generated gerbers, added one missing trace.
Parts:
- removed J3: Prog Jumper, Connector_PinHeader_2.54mm:PinHeader_1x03_P2.54mm_Vertical
- removed R2: 10k, Resistor_SMD:R_0805_2012Metric_Pad1.15x1.40mm_HandSolder
- J1: value Battery Connector -> Battery
- J2: footprint Connector_PinHeader_2.54mm:PinHeader_1x04_P2.54mm_Vertical -> Connector_PinHeader_2.54mm:PinHeader_1x06_P2.54mm_Vertical
- R10, R6, R7: value R_Small -> 330R
- R5: value R_Small -> 150R
- moved R10 39.6 mm to (123.2, 124.0), turned to 90 degrees
- moved J2 37.9 mm to (150.5, 62.3), turned to 0 degrees
- moved R1 9.00 mm to (140.0, 74.2), turned to 180 degrees
- moved C5 1.64 mm to (115.5, 73.4)
- moved C4 1.15 mm to (118.0, 73.4)
- moved C3 0.67 mm to (120.5, 73.4)
Connections:
- J2 pad 1: GND -> +3V3
- J2 pad 2: /Tx -> /~RST
- J2 pad 3: /Rx -> /GPIO0
- J2 pad 4: VCC -> /Tx
- U2 pad 1: Net-(R2-Pad2) -> /~RST
- U2 pad 18: Net-(J3-Pad2) -> /GPIO0
Routing:
- net +3V3: track 249.7 -> 0.00 mm, vias 2 -> 0
- net /GPIO0: track 0.00 -> 60.4 mm
- net Net-(D4-Pad1): track 49.3 -> 5.77 mm
- net /LED_BATT: track 4.45 -> 44.6 mm
- net /Rx: track 6.27 -> 43.9 mm
- net /Tx: track 6.33 -> 43.5 mm
- net GND: track 61.6 -> 32.4 mm, vias 1 -> 6
- net Net-(J3-Pad2): track 28.3 -> 0.00 mm
- net /~RST: track 0.00 -> 24.5 mm
- net VCC: track 40.5 -> 21.0 mm
- net Net-(R8-Pad2): track 57.7 -> 49.0 mm, vias 0 -> 2
- net /BUTTON_SAVE: track 13.3 -> 21.8 mm, vias 0 -> 1
- net Net-(R1-Pad2): track 3.85 -> 11.0 mm
- net /BUTTON_CHANGE: track 13.6 -> 20.1 mm, vias 0 -> 1
- net Net-(R2-Pad2): track 3.85 -> 0.00 mm
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- added copper zone on F.Cu, net +3V3
Other:
- board text added: "+ -"
- board text added: "- Rx Tx 0 R +"
- board text added: "Church Sign Controller Ryan Absher 2020"
- board text added: "JLCJLCJLCJLC"

Commit message: Correction
I didn't realize that you couldn't use GPIO 9 on the ESP-12e. Moved battery LED to GPIO 13.
Parts:
- J1: value Battery -> Battery Connector
- R10, R6, R7: value 330R -> R_Small
- R5: value 150R -> R_Small
Connections:
- U2 pad 11: /LED_BATT -> (no net)
- U2 pad 7: (no net) -> /LED_BATT
Routing:
- net /LED_BATT: track 44.6 -> 60.3 mm
Changed lines of the file:
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@@
     (thickness 1.6)
     (drawings 11)
-    (tracks 114)
+    (tracks 116)
     (zones 0)
     (modules 24)
@@
       (effects (font (size 1 1) (thickness 0.15)))
     )
-    (fp_text value Battery (at 3.25 1.29 90) (layer F.SilkS)
+    (fp_text value "Battery Connector" (at 3.25 1.29 90) (layer F.SilkS)
       (effects (font (size 1 1) (thickness 0.15)))
     )
@@
       (effects (font (size 1 1) (thickness 0.15)))
     )
-    (fp_text value 150R (at 0 1.65) (layer F.SilkS)
+    (fp_text value R_Small (at 0 1.65) (layer F.SilkS)
       (effects (font (size 1 1) (thickness 0.15)))
     )
@@
       (effects (font (size 1 1) (thickness 0.15)))
     )
-    (fp_text value 330R (at 0 1.65) (layer F.SilkS)
+    (fp_text value R_Small (at 0 1.65) (layer F.SilkS)
       (effects (font (size 1 1) (thickness 0.15)))
     )
@@
       (effects (font (size 1 1) (thickness 0.15)))
     )
-    (fp_text value 330R (at 0 1.65) (layer F.SilkS)
+    (fp_text value R_Small (at 0 1.65) (layer F.SilkS)
       (effects (font (size 1 1) (thickness 0.15)))
     )
@@
       (effects (font (size 1 1) (thickness 0.15)))
     )
-    (fp_text value 330R (at -2.725 0) (layer F.SilkS)
+    (fp_text value R_Small (at -2.725 0) (layer F.SilkS)
       (effects (font (size 1 1) (thickness 0.15)))
     )
@@
     (pad 6 smd rect (at -7.6 6.5 270) (size 2.5 1) (layers F.Cu F.Paste F.Mask)
       (net 13 /LED_GREEN))
-    (pad 7 smd rect (at -7.6 8.5 270) (size 2.5 1) (layers F.Cu F.Paste F.Mask))
+    (pad 7 smd rect (at -7.6 8.5 270) (size 2.5 1) (layers F.Cu F.Paste F.Mask)
+      (net 17 /LED_BATT))
     (pad 8 smd rect (at -7.6 10.5 270) (size 2.5 1) (layers F.Cu F.Paste F.Mask)
       (net 3 +3V3))
     (pad 9 smd rect (at -5 12 270) (size 1 1.8) (layers F.Cu F.Paste F.Mask))
     (pad 10 smd rect (at -3 12 270) (size 1 1.8) (layers F.Cu F.Paste F.Mask))
-    (pad 11 smd rect (at -1 12 270) (size 1 1.8) (layers F.Cu F.Paste F.Mask)
-      (net 17 /LED_BATT))
+    (pad 11 smd rect (at -1 12 270) (size 1 1.8) (layers F.Cu F.Paste F.Mask))
     (pad 12 smd rect (at 1 12 270) (size 1 1.8) (layers F.Cu F.Paste F.Mask))
     (pad 13 smd rect (at 3 12 270) (size 1 1.8) (layers F.Cu F.Paste F.Mask))
@@
   (segment (start 134 76) (end 133 77) (width 0.5) (layer F.Cu) (net 16))
   (segment (start 133 77) (end 133 78.9) (width 0.5) (layer F.Cu) (net 16))
-  (segment (start 118.1 85.5) (end 115 88.6) (width 0.5) (layer F.Cu) (net 17))
-  (segment (start 119.5 85.5) (end 118.1 85.5) (width 0.5) (layer F.Cu) (net 17))
-  (segment (start 115 88.6) (end 115 116.5) (width 0.5) (layer F.Cu) (net 17))
-  (segment (start 121.5 123) (end 123.25 123) (width 0.5) (layer F.Cu) (net 17))
-  (segment (start 115 116.5) (end 121.5 123) (width 0.5) (layer F.Cu) (net 17))
+  (segment (start 121 123) (end 123.25 123) (width 0.5) (layer F.Cu) (net 17))
+  (segment (start 123 77) (end 122.5 76.5) (width 0.5) (layer F.Cu) (net 17))
+  (segment (start 123 78.9) (end 123 77) (width 0.5) (layer F.Cu) (net 17))
+  (segment (start 122.5 76.5) (end 117.5 76.5) (width 0.5) (layer F.Cu) (net 17))
+  (segment (start 117.5 76.5) (end 114.5 79.5) (width 0.5) (layer F.Cu) (net 17))
+  (segment (start 114.5 79.5) (end 114.5 116.5) (width 0.5) (layer F.Cu) (net 17))
+  (segment (start 114.5 116.5) (end 121 123) (width 0.5) (layer F.Cu) (net 17))
   (segment (start 140.085787 106) (end 135 106) (width 0.5) (layer B.Cu) (net 18))
   (segment (start 141.5 106) (end 140.085787 106) (width 0.5) (layer B.Cu) (net 18))
